Commit message: fixed collision geometry of poking stick

File: thor_mang_description/urdf/thor_poking_stick.urdf.xacro (robot description, xacro)
@@ -25,7 +25,7 @@
    </visual>
    <collision>
-     <origin xyz="0 0 0" rpy="0 1.57 0"/>
+     <origin xyz="-0.055 0 0" rpy="0 1.57 0"/>
      <geometry>
-       <cylinder radius="0.001" length="0.001"/>
+       <cylinder radius="0.007" length="0.115"/>
      </geometry>
    </collision>

Commit message: Adjusted poking stick model

File: thor_mang_description/urdf/thor_poking_stick.urdf.xacro (robot description, xacro)
@@ -18,5 +18,5 @@
      <origin xyz="-0.055 0 0" rpy="0 1.57 0" />
      <geometry>
-       <cylinder radius="0.007" length="0.115" />
+       <cylinder radius="0.005" length="0.115" />
      </geometry>
      <material name="Cyan">
@@ -27,5 +27,5 @@
      <origin xyz="-0.055 0 0" rpy="0 1.57 0"/>
      <geometry>
-       <cylinder radius="0.007" length="0.115"/>
+       <cylinder radius="0.005" length="0.115"/>
      </geometry>
    </collision>

Commit message: changed name of poking stick frame

File: thor_mang_description/urdf/thor_poking_stick.urdf.xacro (robot description, xacro)
@@ -2,12 +2,12 @@
 <robot  name="thor_poking_stick" xmlns:xacro="http://www.ros.org/wiki/xacro">
   <macro name="thor_poking_stick_macro" params="parent *origin">
-  <joint name="poking_stick_joint" type="fixed">
+  <joint name="left_poking_stick_joint" type="fixed">
     <insert_block name="origin"/>
     <parent
       link="${parent}" />
     <child
-       link="poking_stick"/>
+       link="left_poking_stick_frame"/>
   </joint>
-  <link name="poking_stick">
+  <link name="left_poking_stick_frame">
    <inertial>
      <origin xyz="0.05 0 0" rpy="0 0 0"/>

Commit message: renamed to left_poking_stick

File: thor_mang_description/urdf/thor_poking_stick.urdf.xacro (robot description, xacro)
@@ -7,7 +7,7 @@
       link="${parent}" />
     <child
-       link="left_poking_stick_frame"/>
+       link="left_poking_stick"/>
   </joint>
-  <link name="left_poking_stick_frame">
+  <link name="left_poking_stick">
    <inertial>
      <origin xyz="0.05 0 0" rpy="0 0 0"/>
