Commit message: Moved meshes to new folder for consistency with tud description

File: thor_mang_description/urdf/arm/thor_arm_6dof_simple.urdf.xacro (robot description, xacro)
@@ -37,5 +37,5 @@
       <geometry>
         <mesh
-          filename="package://thor_mang_description/meshes/simple/shoulder_pitch_left.stl" scale="0.001 ${0.001 * reflect} 0.001"/>
+          filename="package://thor_mang_description/meshes/visual/shoulder_pitch_left.stl" scale="0.001 ${0.001 * reflect} 0.001"/>
       </geometry>
       <xacro:black/>
@@ -47,5 +47,5 @@
       <geometry>
         <mesh
-          filename="package://thor_mang_description/meshes/simple/shoulder_pitch_left.stl" scale="0.001 ${0.001 * reflect} 0.001"/>
+          filename="package://thor_mang_description/meshes/visual/shoulder_pitch_left.stl" scale="0.001 ${0.001 * reflect} 0.001"/>
       </geometry>
     </collision>
@@ -76,5 +76,5 @@
       <geometry>
         <mesh
-          filename="package://thor_mang_description/meshes/simple/shoulder_roll_left.stl" scale="0.001 0.001 0.001"/>
+          filename="package://thor_mang_description/meshes/visual/shoulder_roll_left.stl" scale="0.001 0.001 0.001"/>
       </geometry>
       <xacro:black/>
@@ -86,5 +86,5 @@
       <geometry>
         <mesh
-          filename="package://thor_mang_description/meshes/simple/shoulder_roll_left.stl" scale="0.001 0.001 0.001"/>
+          filename="package://thor_mang_description/meshes/visual/shoulder_roll_left.stl" scale="0.001 0.001 0.001"/>
       </geometry>
     </collision>
@@ -114,15 +114,15 @@
       <geometry>
         <mesh
-          filename="package://thor_mang_description/meshes/simple/shoulder_yaw_left.stl" scale="0.001 0.001 0.001"/>
-      </geometry>
-      <xacro:black/>
-    </visual>
-    <collision>
-      <origin
-        xyz="0 0 0"
-        rpy=" ${M_PI*0.5} 0 ${-M_PI*0.5}" />
-      <geometry>
-        <mesh
-          filename="package://thor_mang_description/meshes/simple/shoulder_yaw_left.stl" scale="0.001 0.001 0.001"/>
+          filename="package://thor_mang_description/meshes/visual/shoulder_yaw_left.stl" scale="0.001 0.001 0.001"/>
+      </geometry>
+      <xacro:black/>
+    </visual>
+    <collision>
+      <origin
+        xyz="0 0 0"
+        rpy=" ${M_PI*0.5} 0 ${-M_PI*0.5}" />
+      <geometry>
+        <mesh
+          filename="package://thor_mang_description/meshes/visual/shoulder_yaw_left.stl" scale="0.001 0.001 0.001"/>
       </geometry>
     </collision>
@@ -152,5 +152,5 @@
       <geometry>
         <mesh
-          filename="package://thor_mang_description/meshes/simple/elbow_left.stl" scale="0.001 0.001 0.001"/>
+          filename="package://thor_mang_description/meshes/visual/elbow_left.stl" scale="0.001 0.001 0.001"/>
       </geometry>
       <xacro:black/>
@@ -162,5 +162,5 @@
       <geometry>
         <mesh
-          filename="package://thor_mang_description/meshes/simple/elbow_left.stl" scale="0.001 0.001 0.001"/>
+          filename="package://thor_mang_description/meshes/visual/elbow_left.stl" scale="0.001 0.001 0.001"/>
       </geometry>
     </collision>
@@ -190,15 +190,15 @@
       <geometry>
         <mesh
-          filename="package://thor_mang_description/meshes/simple/wrist_yaw_left.stl" scale="0.001 0.001 0.001"/>
-      </geometry>
-      <xacro:black/>
-    </visual>
-    <collision>
-      <origin
-        xyz="0 0 0"
-        rpy=" ${M_PI*0.5} 0 ${-M_PI*0.5}" />
-      <geometry>
-        <mesh
-          filename="package://thor_mang_description/meshes/simple/wrist_yaw_left.stl" scale="0.001 0.001 0.001"/>
+          filename="package://thor_mang_description/meshes/visual/wrist_yaw_left.stl" scale="0.001 0.001 0.001"/>
+      </geometry>
+      <xacro:black/>
+    </visual>
+    <collision>
+      <origin
+        xyz="0 0 0"
+        rpy=" ${M_PI*0.5} 0 ${-M_PI*0.5}" />
+      <geometry>
+        <mesh
+          filename="package://thor_mang_description/meshes/visual/wrist_yaw_left.stl" scale="0.001 0.001 0.001"/>
       </geometry>
     </collision>
@@ -228,15 +228,15 @@
       <geometry>
         <mesh
-          filename="package://thor_mang_description/meshes/simple/wrist_roll.stl" scale="${-0.001 * reflect} 0.001 0.001"/>
-      </geometry>
-      <xacro:black/>
-    </visual>
-    <collision>
-      <origin
-        xyz="0 0 0"
-        rpy=" ${M_PI*0.5} 0 ${-M_PI*0.5}" />
-      <geometry>
-        <mesh
-          filename="package://thor_mang_description/meshes/simple/wrist_roll.stl" scale="${-0.001 * reflect} 0.001 0.001"/>
+          filename="package://thor_mang_description/meshes/visual/wrist_roll.stl" scale="${-0.001 * reflect} 0.001 0.001"/>
+      </geometry>
+      <xacro:black/>
+    </visual>
+    <collision>
+      <origin
+        xyz="0 0 0"
+        rpy=" ${M_PI*0.5} 0 ${-M_PI*0.5}" />
+      <geometry>
+        <mesh
+          filename="package://thor_mang_description/meshes/visual/wrist_roll.stl" scale="${-0.001 * reflect} 0.001 0.001"/>
       </geometry>
     </collision>

File: thor_mang_description/urdf/arm/thor_arm_7dof_simple.urdf.xacro (robot description, xacro)
@@ -201,5 +201,5 @@
 	<box size="0.035 .035 .01"/>
         <!--<mesh
-          filename="package://thor_mang_description/meshes/simple/wrist_yaw_left.stl" scale="0.001 0.001 0.001"/>-->
+          filename="package://thor_mang_description/meshes/visual/wrist_yaw_left.stl" scale="0.001 0.001 0.001"/>-->
       </geometry>
       <xacro:black/>

File: thor_mang_description/urdf/hands/thor_mang_hand.urdf.xacro (robot description, xacro)
@@ -12,5 +12,5 @@
       <geometry>
         <mesh
-          filename="package://thor_mang_description/meshes/simple/thor_mang_hand.stl" scale="${reflect} 1 1"/>
+          filename="package://thor_mang_description/meshes/visual/thor_mang_hand.stl" scale="${reflect} 1 1"/>
       </geometry>
       <xacro:black/>
@@ -22,5 +22,5 @@
       <geometry>
         <mesh
-          filename="package://thor_mang_description/meshes/simple/thor_mang_hand.stl" scale="${reflect} 1 1"/>
+          filename="package://thor_mang_description/meshes/visual/thor_mang_hand.stl" scale="${reflect} 1 1"/>
       </geometry>
     </collision>
