Commit message: moved r/l_hand frame to hand wrist to make ft sensor simulation in gazebo more accurate

File: thor_mang_description/hands/l_vt_hand.urdf.xacro (robot description, xacro)
@@ -3,5 +3,5 @@
   <xacro:include filename="$(find thor_vt_hand_description)/urdf/vt_hand_tud.urdf.xacro.xml" />
   <vt_hand_tud_macro parent="l_hand" prefix="l" reflect="-1" >
-    <origin xyz="0 0 -0.16" rpy="3.141592 0 1.570796"/>
+    <origin xyz="0 0 -0.015" rpy="3.141592 0 1.570796"/>
   </vt_hand_tud_macro>
 </robot>

File: thor_mang_description/hands/r_vt_hand.urdf.xacro (robot description, xacro)
@@ -3,5 +3,5 @@
   <xacro:include filename="$(find thor_vt_hand_description)/urdf/vt_hand_tud.urdf.xacro.xml" />
   <vt_hand_tud_macro parent="r_hand" prefix="r" reflect="1" >
-    <origin xyz="0 0 -0.16" rpy="3.141592 0 1.570796"/>
+    <origin xyz="0 0 -0.015" rpy="3.141592 0 1.570796"/>
   </vt_hand_tud_macro>
 </robot>

File: thor_mang_description/urdf/arm/thor_arm_7dof_simple.urdf.xacro (robot description, xacro)
@@ -173,5 +173,5 @@
   <joint name="${name}${arm_joint_6_suffix}" type="revolute">
     <origin
-      xyz="0 0 0"
+      xyz="0 0 -0.145"
       rpy="0 0 ${0 + j6_offset}"
        />
@@ -192,9 +192,10 @@
     -->
     <xacro:inertial_cuboid__with_pose_macro mass="0.13" x_length="0.035" y_length="0.035" z_length="0.01">
-      <origin xyz="0.0 0.0 -0.135" rpy="0 0 0"/>
+      <!--<origin xyz="0.0 0.0 -0.135" rpy="0 0 0"/>-->
+      <origin xyz="0 0 0.01" rpy="0 0 0"/>
     </xacro:inertial_cuboid__with_pose_macro>
     <visual>
       <origin
-        xyz="0 0 -0.135"
+        xyz="0 0 0.01"
         rpy=" 0 0 0" />
       <geometry>
